File: board/serial_matrix_keyboard_shild/serial_matrix_keyboard_shild.kicad_pcb (KiCad board)
At the start: 2 copper layers, 27 x 22 mm, 21 parts, among them J1 DATA, J2 AVR-ISP-6, J3 KEYBOARD, U1 ATtiny2313-20SU, Y1 NX3225SA-16.000M-STD-CRS-2

Commit message: Разведена плата.
Parts:
- moved C5 12.3 mm to (201.8, 100.8)
- moved C3 3.57 mm to (216.2, 99.7)
- moved C2 2.88 mm to (220.0, 94.3), turned to 0 degrees
- moved Y1 1.60 mm to (215.2, 95.7)
- moved J2 0.30 mm to (211.8, 104.5)
- moved J3 0.30 mm to (199.3, 87.0)
- moved U1 0.30 mm to (203.4, 96.0)
- moved R1 0.30 mm to (208.1, 100.8)
- moved C1 0.30 mm to (211.2, 102.1)
- moved J1 0.30 mm to (216.8, 104.5)
- turned D5 to 90 degrees
Routing:
- net +5V: track 0.00 -> 55.4 mm, vias 0 -> 1
- net /BC4: track 0.00 -> 27.7 mm, vias 0 -> 1
- net /BC2: track 0.00 -> 17.6 mm, vias 0 -> 1
- net /BR4: track 0.00 -> 16.4 mm, vias 0 -> 1
- net /MISO: track 0.00 -> 16.2 mm
- net /XTAL1: track 0.00 -> 15.7 mm
- net /RESET: track 0.00 -> 15.0 mm, vias 0 -> 1
- net /TX: track 0.00 -> 13.5 mm
- net /BR2: track 0.00 -> 13.4 mm, vias 0 -> 1
- net /BR3: track 0.00 -> 13.3 mm, vias 0 -> 1
- net /BC3: track 0.00 -> 13.0 mm, vias 0 -> 1
- net /MOSI: track 0.00 -> 11.7 mm, vias 0 -> 2
- net /SCK: track 0.00 -> 11.5 mm
- net /BC1: track 0.00 -> 10.8 mm, vias 0 -> 1
- net /BR1: track 0.00 -> 10.3 mm, vias 0 -> 1
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- added copper zone on B.Cu, net GND
- added copper zone on F.Cu, net GND

Commit message: Мелкие правки перед производитсвом и добавлены gerber.
Parts:
- moved C1 0.47 mm to (211.3, 101.7)
Routing:
- net +5V: track 55.4 -> 62.6 mm
- net /BR1: track 10.3 -> 8.97 mm
- net /BR0: track 6.85 -> 6.33 mm
